File: KiCAD/Micro_alimentation.kicad_pcb (KiCad board)
At the start: 4 copper layers, 50 x 70 mm, 38 parts, among them J1 Conn_01x02, J2 Conn_01x02, J3 Piles, J4 Micro, SW1 SW_DIP_x01, U1 Opamp_Dual

Commit message: Update : PCB + bom
Parts:
- added TP1: TestPoint, TestPoint:TestPoint_Bridge_Pitch2.0mm_Drill0.7mm, F.Cu at (62.0, 104.0)
- added TP2: TestPoint, TestPoint:TestPoint_Bridge_Pitch2.0mm_Drill0.7mm, F.Cu at (61.0, 54.0)
- added TP3: TestPoint, TestPoint:TestPoint_Bridge_Pitch2.0mm_Drill0.7mm, F.Cu at (75.0, 104.0)
- added TP4: TestPoint, TestPoint:TestPoint_Bridge_Pitch2.0mm_Drill0.7mm, F.Cu at (66.0, 104.0)
- U1: footprint Package_SO:SOIC-8-1EP_3.9x4.9mm_P1.27mm_EP2.29x3mm_ThermalVias -> Package_SO:SOIC-8_3.9x4.9mm_P1.27mm
Routing:
- net GND: track 185.8 -> 15.4 mm, vias 4 -> 0
- net Net-(J1-Pin_1): track 3.91 -> 8.91 mm
- net Net-(J4-Pin_1): track 11.1 -> 16.1 mm
- net Net-(J2-Pin_1): track 3.89 -> 8.89 mm
- net Net-(D3-A): track 8.09 -> 11.5 mm
- net VCC: track 28.7 -> 26.5 mm
- added copper zone on B.Cu, net GND
- added copper zone on F.Cu, net GND
- removed copper zone on B.Cu, net (none)
- removed copper zone on F.Cu, net (none)
