File: KiCAD/Micro_alimentation.kicad_sch (KiCad schematic)
At the start: 38 parts, among them J1 Conn_01x02, J2 Conn_01x02, J3 Piles, J4 Micro, SW1 SW_DIP_x01, U1 Opamp_Dual

Commit message: Update : PCB + bom
Parts:
- added TP1, TP2, TP3, TP4: TestPoint, TestPoint:TestPoint_Bridge_Pitch2.0mm_Drill0.7mm, symbol Connector:TestPoint
- U1: footprint Package_SO:SOIC-8-1EP_3.9x4.9mm_P1.27mm_EP2.29x3mm_ThermalVias -> Package_SO:SOIC-8_3.9x4.9mm_P1.27mm
Connections:
- net at C10.1, J4.1 (Pin_1), R11.2: now also TP2.1
- net at D3.2 (A), J3.1 (Pin_1): now also TP1.1
- net at J2.1 (Pin_1), R13.2: now also TP3.1
- net at J1.1 (Pin_1), R5.2: now also TP4.1
